Commit message: Controller added for the arm

File: hew/urdf/Actual_HEW.urdf (robot description, URDF)
Before this commit: robot HEW_rob, 3 links, 3 joints
Links:
- link Arm_Link: geometry collision mesh filename=package://hew_description/meshes/Arm_Link_col.STL; visual mesh filename=package://hew/urdf/meshes/Arm_Link.STL

File: hew/urdf/hew_rob.urdf (robot description, URDF)
Before this commit: robot HEW_rob, 2 links, 1 joints
Links:
- added link base_link, mass 2.4395; collision mesh filename=package://hew/urdf/meshes/base_link_col.STL; visual mesh filename=package://hew/urdf/meshes/base_link.STL
Joints:
- removed joint Arm_Link_cont
- added joint fixed: type fixed, parent world, child base_link, origin xyz=0 0 1 rpy=0 3.14 0
- added joint joint1: type continuous, parent base_link, child Arm_Link, origin xyz=0.31115 0.254 -0.084782 rpy=3.1416 0 0, axis 0 0 1
