Commit message: Added horizontal transmission and actuation function

File: hew/urdf/hew_rob.urdf (robot description, URDF)
Before this commit: robot HEW_rob, 3 links, 2 joints
Links:
- added link Horz_Trans, mass 0.015733; collision mesh filename=package://hew/urdf/meshes/Horz_Trans_col.STL; visual mesh filename=package://hew/urdf/meshes/Horz_Trans.STL
Joints:
- added joint joint2: type continuous, parent Arm_Link, child Horz_Trans, origin xyz=-0.10387 0.00038259 -0.0853 rpy=0 0 -0.0036833, axis 1 0 0

Commit message: Joints articulate correclty, contact error present

File: hew/urdf/hew_rob.urdf (robot description, URDF)
Before this commit: robot HEW_rob, 4 links, 3 joints
Links:
- added link Front_Wheel_link, mass 0.33878; collision mesh filename=package://hew/urdf/meshes/Front_Wheel_link_col.STL; visual mesh filename=package://hew/urdf/meshes/Front_Wheel_link.STL
Joints:
- added joint Front_Wheel_cont: type continuous, parent Horz_Trans, child Front_Wheel_link, origin xyz=0.10387 0 0 rpy=0 0 -3.1416, axis 0 0 1
